Commit message: wp0 manipulator description

File: ur_manipulator_description/urdf/base_attachment.urdf.xacro (robot description, xacro)
@@ -1,41 +1,22 @@
 <?xml version="1.0"?>
-<robot xmlns:xacro="http://ros.org/wiki/xacro" name="base_attachment">
-  <!-- Macro for the base attachment using params -->
-  <xacro:macro name="base_attachment" params="name base_parent robot">
-    <!-- Joint to connect cylinder base to the world -->
-    <joint name="${name}_to_world" type="fixed">
-        <parent link="${base_parent}"/>
-        <child link="${name}_base_link"/>
-        <origin xyz="-0.095725 0.65 0.425" rpy="0 0 -1.5708"/> <!-- Lift by half the cylinder height -->
+<robot xmlns:xacro="http://wiki.ros.org/xacro" name="base_attachment">
+  <xacro:macro name="base_attachment" params="name parent">
+    <!-- Fixed joint: parent (e.g., world) -> base platform -->
+    <joint name="${name}_to_${parent}" type="fixed">
+      <parent link="${parent}"/>
+      <child  link="${name}_base_link"/>
+      <origin xyz="-0.095725 0.65 0.425" rpy="0 0 -1.5708"/>
     </joint>
-    <!-- Grey Cylinder Base -->
     <link name="${name}_base_link">
       <visual>
-        <geometry>
-          <cylinder radius="0.1" length="0.85"/>
-        </geometry>
-        <material name="grey">
-          <color rgba="0.5 0.5 0.5 1.0"/>
-        </material>
-        <origin xyz="0 0 0" rpy="0 0 0"/>
+        <geometry><cylinder radius="0.1" length="0.85"/></geometry>
+        <material name="grey"><color rgba="0.5 0.5 0.5 1.0"/></material>
       </visual>
-      <collision>
-        <geometry>
-          <cylinder radius="0.1" length="0.85"/>
-        </geometry>
-        <origin xyz="0 0 0" rpy="0 0 0"/>
-      </collision>
+      <collision><geometry><cylinder radius="0.1" length="0.85"/></geometry></collision>
       <inertial>
         <mass value="10.0"/>
-        <origin xyz="0 0 0" rpy="0 0 0"/>
         <inertia ixx="0.1" ixy="0.0" ixz="0.0" iyy="0.1" iyz="0.0" izz="0.1"/>
       </inertial>
     </link>
-    <!-- Joint between Cylinder Base and UR5 Robot -->
-    <joint name="${name}_to_${robot}" type="fixed">
-      <parent link="${name}_base_link"/>
-      <child link="${robot}_base_link"/> <!-- As per your request -->
-      <origin xyz="0 0 0.425" rpy="0 0 0"/> <!-- Position the UR5 on top of the cylinder -->
-    </joint>
   </xacro:macro>
 </robot>

File: ur_manipulator_description/urdf/manipulator.urdf.xacro (robot description, xacro)
@@ -1,27 +1,21 @@
 <?xml version="1.0"?>
 <robot xmlns:xacro="http://ros.org/wiki/xacro" name="ur3_manipulator">
-    <!-- Define a property to select your robot prefix -->
-    <xacro:property name="robot_prefix" value="ur3" />
-    <!-- Include base attachment -->
-    <!-- <xacro:include filename="$(find ur_manipulator_description)/urdf/base_attachment.urdf.xacro" /> -->
-    <!-- Include UR5 robot from ros_industrial/ur_description -->
-    <xacro:include filename="$(find ur_manipulator_description)/xacro/rbyt_ur_mocked.xacro"/>
-    <!-- Include table macro -->
-    <!-- <xacro:include filename="$(find manipulator_description)/urdf/table/table.urdf.xacro" /> -->
-    <!-- Define the world link -->
-    <!-- <link name="world" /> -->
-    <!-- Call the base attachment using the property value -->
-    <!-- <xacro:base_attachment name="${robot_prefix}_attachment" base_parent="world" robot="${robot_prefix}" /> -->
-    <!-- Call the UR robot using the property value -->
-    <xacro:rbyt_ur_description
+  <xacro:property name="robot_prefix" value="ur3"/>
+  <!-- Global world frame -->
+  <link name="world"/>
+  <!-- Include macros -->
+  <xacro:include filename="$(find ur_manipulator_description)/urdf/base_attachment.urdf.xacro"/>
+  <xacro:include filename="$(find ur_manipulator_description)/xacro/rbyt_ur_mocked.xacro"/>
+  <!-- 1) Place the base/platform -->
+  <xacro:base_attachment name="${robot_prefix}_attachment" parent="world"/>
+  <!-- 2) Mount the UR arm to the base's link -->
+  <xacro:rbyt_ur_description
       name="ur3"
       ur_type="ur3"
-      tf_prefix="ur3"
-      safety_limits="true"
-      safety_pos_margin="0.15"
-      safety_k_position="20"
-      force_abs_paths="false"
-      mock_sensor_commands="false"/>
-    <!-- add table -->
-    <!-- <xacro:table name="table" table_parent="world"/> -->
+      tf_prefix="${robot_prefix}"
+      base_parent="${robot_prefix}_attachment_base_link"
+      safety_limits="true">
+    <!-- optional fine-tuning of robot pose on the base -->
+    <!-- <origin xyz="0 0 0.0" rpy="0 0 0"/> -->
+  </xacro:rbyt_ur_description>
 </robot>

File: ur_manipulator_description/xacro/rbyt_ur_mocked.xacro (robot description, xacro)
@@ -1,8 +1,10 @@
 <?xml version="1.0"?>
 <robot xmlns:xacro="http://wiki.ros.org/xacro">
+  <!-- Wrapper over UR's ur_robot. No <link name="world"/> here. -->
   <xacro:macro name="rbyt_ur_description" params="
       name:=ur
       ur_type:=ur5
       tf_prefix:=
+      base_parent:=world
       safety_limits:=false
       safety_pos_margin:=0.15
@@ -10,9 +12,8 @@
       force_abs_paths:=false
       mock_sensor_commands:=false
+      *ur_origin
   ">
-    <!-- Include vendor macros -->
     <xacro:include filename="$(find ur_description)/urdf/ur_macro.xacro"/>
     <xacro:include filename="$(find ur_description)/urdf/ros2_control_mock_hardware.xacro"/>
-    <!-- Paths derived from ur_type -->
     <xacro:property name="joint_limit_params"     value="$(find ur_description)/config/${ur_type}/joint_limits.yaml"/>
     <xacro:property name="kinematics_params"      value="$(find ur_description)/config/${ur_type}/default_kinematics.yaml"/>
@@ -20,10 +21,9 @@
     <xacro:property name="visual_params"          value="$(find ur_description)/config/${ur_type}/visual_parameters.yaml"/>
     <xacro:property name="initial_positions_file" value="$(find ur_description)/config/initial_positions.yaml"/>
-    <!-- No <link name="world"/> here; caller provides 'parent' -->
-    <link name="world"/>
+    <!-- Mount the UR arm to the caller-provided parent -->
     <xacro:ur_robot
         name="${name}"
         tf_prefix="${tf_prefix}"
-        parent="world"
+        parent="${base_parent}"
         joint_limits_parameters_file="${joint_limit_params}"
         kinematics_parameters_file="${kinematics_params}"
@@ -34,7 +34,8 @@
         safety_k_position="${safety_k_position}"
         force_abs_paths="${force_abs_paths}">
+      <!-- default pose; caller can override with *ur_origin -->
       <origin xyz="0 0 0" rpy="0 0 0"/>
+      <xacro:insert_block name="ur_origin"/>
     </xacro:ur_robot>
-    <!-- ros2_control instance (uses params, not $(arg ...)) -->
     <xacro:ur_ros2_control
       name="${name}"

Commit message: clean urdf build

File: ur_manipulator_description/urdf/base_attachment.urdf.xacro (robot description, xacro)
@@ -1,22 +1,40 @@
 <?xml version="1.0"?>
 <robot xmlns:xacro="http://wiki.ros.org/xacro" name="base_attachment">
-  <xacro:macro name="base_attachment" params="name parent">
-    <!-- Fixed joint: parent (e.g., world) -> base platform -->
-    <joint name="${name}_to_${parent}" type="fixed">
-      <parent link="${parent}"/>
-      <child  link="${name}_base_link"/>
-      <origin xyz="-0.095725 0.65 0.425" rpy="0 0 -1.5708"/>
+  <xacro:macro name="base_attachment" params="name parent robot">
+    <!-- Joint to connect cylinder base to the world -->
+    <joint name="${name}_to_world" type="fixed">
+        <parent link="${parent}"/>
+        <child link="${name}_base_link"/>
+        <origin xyz="0 0 0" rpy="0 0 0"/>
     </joint>
+    <!-- Grey Cylinder Base -->
     <link name="${name}_base_link">
       <visual>
-        <geometry><cylinder radius="0.1" length="0.85"/></geometry>
-        <material name="grey"><color rgba="0.5 0.5 0.5 1.0"/></material>
+        <geometry>
+          <cylinder radius="0.1" length="0.85"/>
+        </geometry>
+        <material name="grey">
+          <color rgba="0.5 0.5 0.5 1.0"/>
+        </material>
+        <origin xyz="0 0 0" rpy="0 0 0"/>
       </visual>
-      <collision><geometry><cylinder radius="0.1" length="0.85"/></geometry></collision>
+      <collision>
+        <geometry>
+          <cylinder radius="0.1" length="0.85"/>
+        </geometry>
+        <origin xyz="0 0 0" rpy="0 0 0"/>
+      </collision>
       <inertial>
         <mass value="10.0"/>
+        <origin xyz="0 0 0" rpy="0 0 0"/>
         <inertia ixx="0.1" ixy="0.0" ixz="0.0" iyy="0.1" iyz="0.0" izz="0.1"/>
       </inertial>
     </link>
+    <!-- Joint between Cylinder Base and UR5 Robot -->
+    <joint name="${name}_to_${robot}" type="fixed">
+      <parent link="${name}_base_link"/>
+      <child link="${robot}base_link"/> <!-- As per your request -->
+      <origin xyz="0 0 2" rpy="0 0 0"/> <!-- Position the UR5 on top of the cylinder -->
+    </joint>
   </xacro:macro>
 </robot>

File: ur_manipulator_description/urdf/manipulator.urdf.xacro (robot description, xacro)
@@ -1,5 +1,7 @@
 <?xml version="1.0"?>
-<robot xmlns:xacro="http://ros.org/wiki/xacro" name="ur3_manipulator">
-  <xacro:property name="robot_prefix" value="ur3_"/>
+<robot xmlns:xacro="http://ros.org/wiki/xacro" name="ur_manipulator">
+<!-- just set property like in example, possible values: ur3, ur3e, ur5, ur5e, ur7e, ur10, ur10e, ur12e, ur16e, ur15, ur20, ur30 -->
+  <xacro:property name="robot_prefix" value="ur3_"/>    <!-- "example ur3_" -->
+  <xacro:property name="ur_name" value="ur3"/>          <!-- "example ur3" -->
   <!-- Global world frame -->
   <link name="world"/>
@@ -8,11 +10,12 @@
   <xacro:include filename="$(find ur_manipulator_description)/xacro/rbyt_ur_mocked.xacro"/>
   <!-- 1) Place the base/platform -->
-  <xacro:base_attachment name="${robot_prefix}attachment" parent="world"/>
+  <xacro:base_attachment name="${robot_prefix}attachment" parent="world" robot="${robot_prefix}" />
   <!-- 2) Mount the UR arm to the base's link -->
   <xacro:rbyt_ur_description
-      name="ur3"
-      ur_type="ur3"
+      name="${ur_name}"
+      ur_type="${ur_name}"
       tf_prefix="${robot_prefix}"
-      safety_limits="true">
+      ur_parent="${ur_name}_attachment_base_link"
+      safety_limits="false">
   </xacro:rbyt_ur_description>
 </robot>

File: ur_manipulator_description/xacro/rbyt_ur_mocked.xacro (robot description, xacro)
@@ -5,6 +5,6 @@
       name:=ur
       ur_type:=ur5
-      tf_prefix:=
-      base_parent:=world
+      tf_prefix:=ur5_
+      ur_parent:= ur5_attachment_base_link
       safety_limits:=false
       safety_pos_margin:=0.15
@@ -24,5 +24,5 @@
         name="${name}"
         tf_prefix="${tf_prefix}"
-        parent="ur3_attachment_base_link"
+        parent="${ur_parent}"
         joint_limits_parameters_file="${joint_limit_params}"
         kinematics_parameters_file="${kinematics_params}"

Commit message: wp1 manipulator description

File: ur_manipulator_description/urdf/base_attachment.urdf.xacro (robot description, xacro)
@@ -1,26 +1,23 @@
 <?xml version="1.0"?>
 <robot xmlns:xacro="http://wiki.ros.org/xacro" name="base_attachment">
-  <xacro:macro name="base_attachment" params="name parent robot">
-    <!-- Joint to connect cylinder base to the world -->
-    <joint name="${name}_to_world" type="fixed">
-        <parent link="${parent}"/>
-        <child link="${name}_base_link"/>
-        <origin xyz="0 0 0" rpy="0 0 0"/>
+  <!-- name: prefix for this base, parent: link to mount to (e.g., world)
+       height: cylinder length (for convenience), mount_offset: distance from
+       cylinder center to its top; defaults to height/2 -->
+  <xacro:macro name="base_attachment" params="name parent">
+    <!-- Fix the base to the given parent -->
+    <joint name="${name}_to_${parent}" type="fixed">
+      <parent link="${parent}"/>
+      <child  link="${name}_base_link"/>
+      <origin xyz="0 0 0" rpy="0 0 0"/>
     </joint>
-    <!-- Grey Cylinder Base -->
+    <!-- Cylinder base -->
     <link name="${name}_base_link">
       <visual>
-        <geometry>
-          <cylinder radius="0.1" length="0.85"/>
-        </geometry>
-        <material name="grey">
-          <color rgba="0.5 0.5 0.5 1.0"/>
-        </material>
+        <geometry><cylinder radius="0.1" length="0.85"/></geometry>
+        <material name="grey"><color rgba="0.5 0.5 0.5 1.0"/></material>
         <origin xyz="0 0 0" rpy="0 0 0"/>
       </visual>
       <collision>
-        <geometry>
-          <cylinder radius="0.1" length="0.85"/>
-        </geometry>
+        <geometry><cylinder radius="0.1" length="0.85"/></geometry>
         <origin xyz="0 0 0" rpy="0 0 0"/>
       </collision>
@@ -31,9 +28,12 @@
       </inertial>
     </link>
-    <!-- Joint between Cylinder Base and UR5 Robot -->
-    <joint name="${name}_to_${robot}" type="fixed">
+    <!-- Mount link ABOVE the cylinder (no <origin> inside link!) -->
+    <link name="${name}_mount_link"/>
+    <!-- Fixed transform: base_link -> mount_link at the top face -->
+    <joint name="${name}_base_to_mount" type="fixed">
       <parent link="${name}_base_link"/>
-      <child link="${robot}base_link"/> <!-- As per your request -->
-      <origin xyz="0 0 2" rpy="0 0 0"/> <!-- Position the UR5 on top of the cylinder -->
+      <child  link="${name}_mount_link"/>
+      <!-- If height=0.85, top is +0.425 from center -->
+      <origin xyz="0 0 0.425" rpy="0 0 0"/>
     </joint>
   </xacro:macro>

File: ur_manipulator_description/urdf/manipulator.urdf.xacro (robot description, xacro)
@@ -1,7 +1,11 @@
 <?xml version="1.0"?>
 <robot xmlns:xacro="http://ros.org/wiki/xacro" name="ur_manipulator">
+<!-- ########################################################################################################################### -->
 <!-- just set property like in example, possible values: ur3, ur3e, ur5, ur5e, ur7e, ur10, ur10e, ur12e, ur16e, ur15, ur20, ur30 -->
-  <xacro:property name="robot_prefix" value="ur3_"/>    <!-- "example ur3_" -->
-  <xacro:property name="ur_name" value="ur3"/>          <!-- "example ur3" -->
+<!-- ########################################################################################################################### -->
+  <xacro:property name="robot_prefix" value="ur30_"/>    <!-- "example ur3_" -->
+  <xacro:property name="ur_name" value="ur30"/>          <!-- "example ur3" -->
+<!-- ########################################################################################################################### -->
+<!-- ########################################################################################################################### -->
   <!-- Global world frame -->
   <link name="world"/>
@@ -10,5 +14,5 @@
   <xacro:include filename="$(find ur_manipulator_description)/xacro/rbyt_ur_mocked.xacro"/>
   <!-- 1) Place the base/platform -->
-  <xacro:base_attachment name="${robot_prefix}attachment" parent="world" robot="${robot_prefix}" />
+  <xacro:base_attachment name="${robot_prefix}attachment" parent="world" />
   <!-- 2) Mount the UR arm to the base's link -->
   <xacro:rbyt_ur_description
@@ -16,5 +20,5 @@
       ur_type="${ur_name}"
       tf_prefix="${robot_prefix}"
-      ur_parent="${ur_name}_attachment_base_link"
+      ur_parent="${robot_prefix}attachment_mount_link"
       safety_limits="false">
   </xacro:rbyt_ur_description>

File: ur_manipulator_description/xacro/rbyt_ur_mocked.xacro (robot description, xacro)
@@ -6,5 +6,5 @@
       ur_type:=ur5
       tf_prefix:=ur5_
-      ur_parent:= ur5_attachment_base_link
+      ur_parent:= ur5_mount_link
       safety_limits:=false
       safety_pos_margin:=0.15
