Commit message: successfull urdf build

File: ur_manipulator_description/urdf/manipulator.urdf.xacro (robot description, xacro)
@@ -1,5 +1,5 @@
 <?xml version="1.0"?>
 <robot xmlns:xacro="http://ros.org/wiki/xacro" name="ur3_manipulator">
-  <xacro:property name="robot_prefix" value="ur3"/>
+  <xacro:property name="robot_prefix" value="ur3_"/>
   <!-- Global world frame -->
   <link name="world"/>
@@ -8,5 +8,5 @@
   <xacro:include filename="$(find ur_manipulator_description)/xacro/rbyt_ur_mocked.xacro"/>
   <!-- 1) Place the base/platform -->
-  <xacro:base_attachment name="${robot_prefix}_attachment" parent="world"/>
+  <xacro:base_attachment name="${robot_prefix}attachment" parent="world"/>
   <!-- 2) Mount the UR arm to the base's link -->
   <xacro:rbyt_ur_description
@@ -14,8 +14,5 @@
       ur_type="ur3"
       tf_prefix="${robot_prefix}"
-      base_parent="${robot_prefix}_attachment_base_link"
       safety_limits="true">
-    <!-- optional fine-tuning of robot pose on the base -->
-    <!-- <origin xyz="0 0 0.0" rpy="0 0 0"/> -->
   </xacro:rbyt_ur_description>
 </robot>

File: ur_manipulator_description/xacro/rbyt_ur_mocked.xacro (robot description, xacro)
@@ -12,5 +12,4 @@
       force_abs_paths:=false
       mock_sensor_commands:=false
-      *ur_origin
   ">
     <xacro:include filename="$(find ur_description)/urdf/ur_macro.xacro"/>
@@ -25,5 +24,5 @@
         name="${name}"
         tf_prefix="${tf_prefix}"
-        parent="${base_parent}"
+        parent="ur3_attachment_base_link"
         joint_limits_parameters_file="${joint_limit_params}"
         kinematics_parameters_file="${kinematics_params}"
@@ -34,7 +33,5 @@
         safety_k_position="${safety_k_position}"
         force_abs_paths="${force_abs_paths}">
-      <!-- default pose; caller can override with *ur_origin -->
       <origin xyz="0 0 0" rpy="0 0 0"/>
-      <xacro:insert_block name="ur_origin"/>
     </xacro:ur_robot>
     <xacro:ur_ros2_control

Commit message: wp2 manipulator description

File: ur_manipulator_description/urdf/manipulator.urdf.xacro (robot description, xacro)
@@ -1,11 +1,11 @@
 <?xml version="1.0"?>
 <robot xmlns:xacro="http://ros.org/wiki/xacro" name="ur_manipulator">
-<!-- ########################################################################################################################### -->
-<!-- just set property like in example, possible values: ur3, ur3e, ur5, ur5e, ur7e, ur10, ur10e, ur12e, ur16e, ur15, ur20, ur30 -->
-<!-- ########################################################################################################################### -->
-  <xacro:property name="robot_prefix" value="ur30_"/>    <!-- "example ur3_" -->
-  <xacro:property name="ur_name" value="ur30"/>          <!-- "example ur3" -->
-<!-- ########################################################################################################################### -->
-<!-- ########################################################################################################################### -->
+  <!-- ########################################################################################################################### -->
+  <!-- just set property like in example, possible values: ur3, ur3e, ur5, ur5e, ur7e, ur10, ur10e, ur12e, ur16e, ur15, ur20, ur30 -->
+  <!-- ########################################################################################################################### -->
+  <xacro:property name="robot_prefix" value="ur3_"/>    <!-- "example ur3_" -->
+  <xacro:property name="ur_name" value="ur3"/>          <!-- "example ur3" -->
+  <!-- ########################################################################################################################### -->
+  <!-- ########################################################################################################################### -->
   <!-- Global world frame -->
   <link name="world"/>
